Commit message: Añadido modelo de robot de 4 ruedas. Localización del robot implementada

File: camera_description/urdf/camera.urdf (robot description, URDF)
Before this commit: robot CPRcamera, 3 links, 2 joints
Joints:
- joint fixed: origin xyz=0 0 0 rpy=0 1.570796327 0 -> xyz=0 0 0 rpy=0 1.570796327 1.570796327
